File: KiCAD/antenna_analyzer_v1.kicad_pcb (KiCad board)
At the start: 2 copper layers, 26 parts, among them P1 CONN_01X02, P2 CONN_01X02, P3 CONN_01X02, P4 CONN_01X04, P5 CONN_01X03, P6 CONN_01X02, U1 MCP6002

Commit message: Latest changes to pcb files
Parts:
- added J1: RFTEST, SMA-edge:Molex_SMA_Jack_Edge_Mount, F.Cu at (101.0, 79.5)
- added J2: DUT, SMA-edge:Molex_SMA_Jack_Edge_Mount, F.Cu at (139.0, 79.5)
- C1: value 1u -> 0.01u; footprint Capacitors_THT:C_Disc_D7.5mm_W5.0mm_P5.00mm -> Capacitors_THT:C_Disc_D4.7mm_W2.5mm_P5.00mm; moved to B.Cu
- C2: value 0.1u -> 1u; footprint Capacitors_THT:C_Disc_D7.5mm_W5.0mm_P5.00mm -> Capacitors_THT:C_Disc_D4.7mm_W2.5mm_P5.00mm; moved to B.Cu
- C3: footprint Capacitors_THT:C_Disc_D7.5mm_W5.0mm_P5.00mm -> Capacitors_THT:C_Disc_D4.7mm_W2.5mm_P5.00mm
- C4: value 0.01u -> 0.1u; footprint Capacitors_THT:C_Disc_D7.5mm_W5.0mm_P5.00mm -> Capacitors_THT:C_Disc_D4.7mm_W2.5mm_P5.00mm; moved to B.Cu
- C5: footprint Capacitors_THT:C_Disc_D7.5mm_W5.0mm_P5.00mm -> Capacitors_THT:C_Disc_D4.7mm_W2.5mm_P5.00mm; moved to B.Cu
- C6: value C_Small -> 0.01u; footprint Capacitors_THT:C_Disc_D7.5mm_W5.0mm_P5.00mm -> Capacitors_THT:C_Disc_D4.7mm_W2.5mm_P5.00mm; moved to B.Cu
- D1, D2: footprint Diodes_THT:D_A-405_P12.70mm_Horizontal -> Diodes_THT:D_5W_P12.70mm_Horizontal; moved to B.Cu
- P1, P2, P3: moved to B.Cu
- P4: value CONN_01X04 -> CONN_01X02; footprint Pin_Headers:Pin_Header_Straight_1x04 -> Pin_Headers:Pin_Header_Straight_1x02; moved to B.Cu
- P5: value CONN_01X03 -> CONN_01X04; footprint Pin_Headers:Pin_Header_Straight_1x03 -> Pin_Headers:Pin_Header_Straight_1x04; moved to B.Cu
- P6: value CONN_01X02 -> CONN_01X03; footprint Pin_Headers:Pin_Header_Straight_1x02 -> Pin_Headers:Pin_Header_Straight_1x03; moved to B.Cu
- R1, R10, R11, R2, R3, R4, R5, R6, R7, R8, R9: footprint Resistors_ThroughHole:Resistor_Horizontal_RM15mm -> Resistors_THT:R_Axial_DIN0207_L6.3mm_D2.5mm_P10.16mm_Horizontal; moved to B.Cu
- U1: footprint Housings_DIP:DIP-8_W7.62mm -> Housings_DIP:DIP-8_W7.62mm_Socket; moved to B.Cu
- moved P1 111.9 mm to (101.0, 85.0), turned to 90 degrees
- moved C6 111.5 mm to (98.0, 98.8)
- moved C1 107.6 mm to (111.8, 98.8), turned to 90 degrees
- moved P5 101.8 mm to (124.2, 94.2), turned to 90 degrees
- moved P2 100.0 mm to (127.0, 82.0), turned to 270 degrees
- moved C4 99.7 mm to (103.0, 90.0), turned to 180 degrees
- moved P6 86.1 mm to (118.7, 110.0), turned to 270 degrees
- moved C2 86.0 mm to (110.0, 85.0), turned to 180 degrees
- moved C3 83.2 mm to (136.5, 85.5), turned to 180 degrees
- moved P3 80.7 mm to (113.0, 77.5), turned to 90 degrees
- moved R2 79.3 mm to (119.5, 78.0)
- moved U1 75.8 mm to (123.8, 98.6), turned to 180 degrees
- moved C5 74.0 mm to (137.4, 103.6), turned to 270 degrees
- moved R3 68.0 mm to (113.0, 85.0)
- moved R7 66.8 mm to (97.8, 102.8), turned to 270 degrees
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Connections:
- C1 pad 1: Net-(C1-Pad1) -> +5V
- C1 pad 2: Net-(C1-Pad2) -> GND
- C3 pad 2: GND -> Net-(C3-Pad2)
- C6 pad 1: GND -> Net-(C6-Pad1)
- C6 pad 2: +5V -> GND
- D1 pad 1: Net-(C2-Pad2) -> Net-(C3-Pad2)
- D2 pad 1: Net-(C3-Pad1) -> Net-(C4-Pad1)
- P1 pad 1: Net-(C1-Pad2) -> Net-(C2-Pad2)
- P2 pad 1: Net-(C1-Pad1) -> Net-(D1-Pad2)
- P4 pad 1: +5V -> Net-(C3-Pad1)
- P4 pad 2: /Vrev -> GND
- P5 pad 2: GND -> /Vrev
- P5 pad 3: GND -> /Vfwd
- P6 pad 1: Net-(D1-Pad2) -> GND
- R1 pad 1: Net-(C1-Pad1) -> Net-(C2-Pad1)
- R3 pad 1: Net-(C1-Pad1) -> Net-(C2-Pad1)
- R3 pad 2: Net-(C2-Pad1) -> Net-(C3-Pad1)
- R4 pad 1: Net-(C4-Pad1) -> Net-(C5-Pad1)
- R4 pad 2: Net-(C2-Pad2) -> Net-(C3-Pad2)
- R5 pad 1: Net-(C5-Pad1) -> Net-(C6-Pad1)
- R5 pad 2: Net-(C3-Pad1) -> Net-(C4-Pad1)
- R6 pad 1: Net-(C4-Pad1) -> Net-(C5-Pad1)
- R7 pad 1: Net-(C5-Pad1) -> Net-(C6-Pad1)
- U1 pad 3: Net-(C4-Pad1) -> Net-(C5-Pad1)
- U1 pad 4: (no net) -> GND
- U1 pad 5: Net-(C5-Pad1) -> Net-(C6-Pad1)
- U1 pad 8: (no net) -> +5V
Routing:
- net Net-(C1-Pad1): track 248.3 -> 0.00 mm, vias 7 -> 0
- net GND: track 193.5 -> 16.1 mm, vias 1 -> 0
- net /Vfwd: track 138.5 -> 13.9 mm, vias 4 -> 0
- net Net-(C4-Pad1): track 94.6 -> 9.36 mm, vias 2 -> 0
- net Net-(C2-Pad2): track 83.9 -> 11.2 mm
- net Net-(C5-Pad1): track 94.2 -> 22.2 mm, vias 1 -> 0
- net Net-(D1-Pad2): track 95.1 -> 23.7 mm
- net /Vrev: track 70.4 -> 13.9 mm
- net Net-(R11-Pad1): track 72.4 -> 16.2 mm
- net Net-(C3-Pad1): track 82.6 -> 27.4 mm, vias 2 -> 0
- net Net-(R10-Pad1): track 67.9 -> 17.8 mm
- net +5V: track 44.1 -> 9.04 mm
- net Net-(C6-Pad1): track 0.00 -> 30.9 mm
- net Net-(C2-Pad1): track 37.9 -> 10.5 mm
- net Net-(C1-Pad2): track 26.5 -> 0.00 mm
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- added copper zone on F.Cu, net GND
Other:
- board outline added: 50 x 40 mm
- board text added: "José Carlos Ferreira"
