File: KiCAD/antenna_analyzer_v1.sch (KiCad schematic (older format))
At the start: 45 parts

Commit message: latest updates
Parts:
- removed C? (x5): 0.1u, symbol _passive:C
- removed C? (x2): 4.7u, symbol _passive:C
- removed C?: 1u, symbol _passive:C
- removed D?: SP0503BAHT, TO_SOT_Packages_SMD:SOT-143, symbol ESD_Protection:SP0503BAHT
- removed F?: Fuse, symbol device:Fuse
- removed J?: CONN-10033526-N3212LF, conn-fci:CONN-10033526-N3212LF, symbol conn-fci:CONN-10033526-N3212LF
- removed J?: UART, symbol Connector:Conn_01x04
- removed J?: ICP, symbol Connector:Conn_02x03_Counter_Clockwise
- removed J?: LCD, symbol Connector:Conn_02x06_Counter_Clockwise
- removed Q?: 2N7000, TO_SOT_Packages_THT:TO-92_Molded_Narrow, symbol Transistor:2N7000
- removed R? (x2): 10k, symbol _passive:R
- removed RV?: 20k, symbol _passive:POT
- removed TP?: REV, conn-test:TEST-SMD-SMALL, symbol pcb:TESTPOINT
- removed TP?: FWD, conn-test:TEST-SMD-SMALL, symbol pcb:TESTPOINT
- removed U?: DDS_AD9850_CN_DIL, symbol rf_modules:DDS_AD9850_CN_DIL
- removed U?: CP2104, IPC7351-Nominal:PQFN50P400X400X100-25, symbol silabs:CP2104
- removed U?: ATMEGA328-AU, IPC7351-Nominal:QFP80P900X900X120-32, symbol Atmel:ATMEGA328-AU
- added C6: C_Small, Capacitors_SMD:c_elec_5x5.7, symbol C_Small
- added P1, P2, P3, P6: CONN_01X02, Pin_Headers:Pin_Header_Straight_1x02, symbol CONN_01X02
- added P4: CONN_01X04, Pin_Headers:Pin_Header_Straight_1x04, symbol CONN_01X04
- added P5: CONN_01X03, Pin_Headers:Pin_Header_Straight_1x03, symbol CONN_01X03
- C1, C2, C3, C4, C5: renamed from C?; footprint (none) -> Capacitors_THT:C_Disc_D4.7mm_W2.5mm_P5.00mm
- D1, D2: renamed from D?; footprint (none) -> Diodes_THT:D_5W_P12.70mm_Horizontal
- R1, R10, R11, R2, R3, R4, R5, R6, R7, R8, R9: renamed from R?; footprint (none) -> Resistors_ThroughHole:Resistor_Ceramic_Horizontal_L19mm-W8mm-H8mm-p25mm
- gave numbers to parts that had none: 3
Connections:
- net labels added: +5V
- net labels removed: +5, DDS_DATA, DDS_FQUD, DDS_RESET, DDS_WCLK, LCD_BACKLIGHT, LCD_DATA0, LCD_DATA1, LCD_DATA2, LCD_DATA3, LCD_E, LCD_ENABLE, LCD_RS, LCD_RW, PC2uC, uC2PC, uC_RESET
- wire segments 167 -> 68
- no-connect marks 25 -> 0
Other:
- note removed: "DDS"
- note removed: "Only populate\nfor programming"

Commit message: Latest changes to pcb files
Parts:
- removed C6: C_Small, Capacitors_SMD:c_elec_5x5.7, symbol C_Small
- added C1: 0.01u, Capacitors_THT:C_Disc_D4.7mm_W2.5mm_P5.00mm, symbol _passive:C
- added unit 3 of U1
- J1: footprint conn-linx:CONN-CONSMA001 -> SMA-edge:Molex_SMA_Jack_Edge_Mount
- J2: footprint (none) -> SMA-edge:Molex_SMA_Jack_Edge_Mount
- R1, R10, R11, R2, R3, R4, R5, R6, R7, R8, R9: footprint Resistors_ThroughHole:Resistor_Ceramic_Horizontal_L19mm-W8mm-H8mm-p25mm -> Resistors_THT:R_Axial_DIN0207_L6.3mm_D2.5mm_P10.16mm_Horizontal
- U1: footprint dip-sip:DIP-8 -> Housings_DIP:DIP-8_W7.62mm_Socket
- renumbered C1 to C2, C2 to C3, C3 to C4, C4 to C5, C5 to C6, P6 to P2, P2 to P3, P3 to P4, P4 to P5, P5 to P6
Connections:
- wire segments 68 -> 69
