File: KiCAD/uCLCD/uCLCD.sch (KiCad schematic (older format))
At the start: 17 parts, among them IC1 ATMEGA328P-P, P1 CONN_01X12, P2 CONN_01X03, P3 CONN_01X03, P4 CONN_01X03, P5 CONN_01X02, P6 CONN_01X04, SW1 SW_Push, SW2 SW_Push, SW3 SW_Push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

Commit message: Latest changes to 2nd pcb
Parts:
- removed P6: CONN_01X04, Pin_Headers:Pin_Header_Straight_1x04, symbol CONN_01X04
- removed SW1, SW2, SW3: SW_Push, symbol SW_Push
- added P6: CONN_01X03, Pin_Headers:Pin_Header_Straight_1x03, symbol CONN_01X03
- added P7, P8, P9: p_button, uCLCD:p_button, symbol p_button
- added U1: DDS, uCLCD:DDS9850, symbol DDS
- RV1: footprint Resistors_ThroughHole:Resistor_Horizontal_RM7mm -> Potentiometers:Potentiometer_VishaySpectrol_248GJ_249GJ_Vertical
Connections:
- net +5V: now also U1.1 (Vcc)
- net GND: now also P6.1 (P1), P7.2 (Vcc), P8.2 (Vcc), P9.2 (Vcc), U1.20 (GND), U1.6 (GND)
- net at IC1.1 ((PCINT14/~RESET~)PC6), R1.1: now also P9.1 (GND)
- net at IC1.25 ((PCINT10/ADC2)PC2): now also U1.2 (W_CLK)
- net at IC1.26 ((PCINT11/ADC3)PC3): now also U1.3 (FU_UD)
- net at IC1.27 ((PCINT12/SDA/ADC4)PC4): now also U1.4 (DATA)
- net at IC1.28 ((PCINT13/SCL/ADC5)PC5): now also U1.5 (~RESET)
- net at IC1.4 ((PCINT18/INT0)PD2), R3.1: now also P8.1 (GND)
- net at IC1.5 ((PCINT19/OC2B/INT1)PD3), R2.1: now also P7.1 (GND)
- new net: P6.3 (P3), U1.10 (ZOUT2)
- new net: P6.2 (P2), U1.9 (ZOUT1)
- no-connect marks 3 -> 20
Other:
- moved on the sheet: R2

Commit message: latest changes
Parts:
- P7, P8, P9: footprint uCLCD:p_button -> Buttons_Switches_ThroughHole:SW_PUSH_6mm_h7.3mm
- R1, R2, R3: footprint Resistors_ThroughHole:Resistor_Horizontal_RM7mm -> Resistors_THT:R_Axial_DIN0207_L6.3mm_D2.5mm_P10.16mm_Horizontal
- RV1: footprint Potentiometers:Potentiometer_VishaySpectrol_248GJ_249GJ_Vertical -> Potentiometers:Potentiometer_Trimmer_ACP_CA6v_Horizontal
Connections:
- net +5V: now also R1.1, R2.1, R3.1; no longer R1.2, R2.2, R3.2
- net GND: now also P7.1 (GND), P8.1 (GND), P9.1 (GND); no longer P7.2 (Vcc), P8.2 (Vcc), P9.2 (Vcc)
- net at IC1.13 ((PCINT23/AIN1)PD7): now also P1.4 (P4); no longer P1.5 (P5)
- net at IC1.14 ((PCINT0/CLKO/ICP1)PB0): now also P1.5 (P5); no longer P1.4 (P4)
- net at IC1.25 ((PCINT10/ADC2)PC2): now also U1.5 (~RESET); no longer U1.2 (W_CLK)
- net at IC1.26 ((PCINT11/ADC3)PC3): now also U1.4 (DATA); no longer U1.3 (FU_UD)
- net at IC1.27 ((PCINT12/SDA/ADC4)PC4): now also U1.3 (FU_UD); no longer U1.4 (DATA)
- net at IC1.28 ((PCINT13/SCL/ADC5)PC5): now also U1.2 (W_CLK); no longer U1.5 (~RESET)
- new net: IC1.1 ((PCINT14/~RESET~)PC6), P9.2 (Vcc), R1.2
- new net: IC1.4 ((PCINT18/INT0)PD2), P8.2 (Vcc), R3.2
- new net: IC1.5 ((PCINT19/OC2B/INT1)PD3), P7.2 (Vcc), R2.2
Other:
- note added: "Reset"
- moved on the sheet: P2, P7, R1, R2, R3
