File: KiCAD/uCLCD/uCLCD.kicad_pcb (KiCad board)
At the start: 2 copper layers, 18 parts, among them IC1 ATMEGA328P-P, P1 CONN_01X12, P2 CONN_01X03, P3 CONN_01X03, P4 CONN_01X03, P5 CONN_01X02, P6 CONN_01X03, P7 p_button, P8 p_button, P9 p_button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

Commit message: Latest changes
Parts:
- moved Y1 8.95 mm to (133.8, 73.7)
Changed lines of the file:
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@@
     (links 56)
     (no_connects 56)
-    (area 116.119 23.904999 201.989 98.999)
+    (area 0 0 0 0)
     (thickness 1.6)
     (drawings 0)
@@
   )
   (module Crystals:Crystal_HC49-U_Vertical (layer F.Cu)
-    (at 133.604 64.77 270)
+    (at 133.8 73.72 270)
     (descr "Crystal THT HC-49/U http://5hertz.com/pdfs/04404_D.pdf")
     (tags "THT crystalHC-49/U")
@@
       (effects (font (size 1 1) (thickness 0.15)))
     )
-    (fp_text user %R (at 2.44 0 270) (layer F.Fab)
-      (effects (font (size 1 1) (thickness 0.15)))
-    )
+    (fp_text user %R (at 2.63 -0.196 270) (layer F.Fab)
+      (effects (font (size 1 1) (thickness 0.15)))
+    )
